Commit message: Modified the URDF

File: urdf/barista_robot_model.urdf (robot description, URDF)
Before this commit: robot barista, 16 links, 15 joints
Links:
- removed link standoff_rod_xnyn
- removed link standoff_rod_xnyp
- removed link standoff_rod_xpyn
- removed link standoff_rod_xpyp
- added link standoff_rod_back_left, mass 0.2; collision cylinder length=0.220 radius=0.010; visual cylinder length=0.220 radius=0.010
- added link standoff_rod_back_right, mass 0.2; collision cylinder length=0.220 radius=0.010; visual cylinder length=0.220 radius=0.010
- added link standoff_rod_front_left, mass 0.2; collision cylinder length=0.220 radius=0.010; visual cylinder length=0.220 radius=0.010
- added link standoff_rod_front_right, mass 0.2; collision cylinder length=0.220 radius=0.010; visual cylinder length=0.220 radius=0.010
Joints:
- removed joint standoff_rod_xnyn_joint
- removed joint standoff_rod_xnyp_joint
- removed joint standoff_rod_xpyn_joint
- removed joint standoff_rod_xpyp_joint
- added joint standoff_rod_back_left_joint: type fixed, parent chassis, child standoff_rod_back_left, origin xyz=-0.09 0.09 0.1875 rpy=0 0 0
- added joint standoff_rod_back_right_joint: type fixed, parent chassis, child standoff_rod_back_right, origin xyz=-0.09 -0.09 0.1875 rpy=0 0 0
- added joint standoff_rod_front_left_joint: type fixed, parent chassis, child standoff_rod_front_left, origin xyz=0.09 0.09 0.1875 rpy=0 0 0
- added joint standoff_rod_front_right_joint: type fixed, parent chassis, child standoff_rod_front_right, origin xyz=0.09 -0.09 0.1875 rpy=0 0 0

Commit message: Added frame id into lidar plugin

File: urdf/barista_robot_model.urdf (robot description, URDF)
Before this commit: robot barista_robot, 16 links, 15 joints
Joints:
- joint laser_model_link_joint: origin xyz=0.120 0.0 +0.1275 rpy=0 0 0 -> xyz=0.120 0.0 0.1275 rpy=0 0 0
- joint standoff_rod_back_left_joint: origin xyz=-0.09 0.09 0.1875 rpy=0 0 0 -> xyz=-0.04 0.12 0.1875 rpy=0 0 0
- joint standoff_rod_back_right_joint: origin xyz=-0.09 -0.09 0.1875 rpy=0 0 0 -> xyz=-0.04 -0.12 0.1875 rpy=0 0 0
- joint standoff_rod_front_left_joint: origin xyz=0.09 0.09 0.1875 rpy=0 0 0 -> xyz=0.04 0.12 0.1875 rpy=0 0 0
- joint standoff_rod_front_right_joint: origin xyz=0.09 -0.09 0.1875 rpy=0 0 0 -> xyz=0.04 -0.12 0.1875 rpy=0 0 0

Commit message: Modified collision and number of rays samples

File: urdf/barista_robot_model.urdf (robot description, URDF)
Before this commit: robot barista_robot, 16 links, 15 joints
Links:
- link laser_model: geometry collision cylinder length=0.040 radius=0.03; visual mesh filename=package://barista_robot_description/meshes/hokuyo_urg_04lx.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
Joints:
- joint standoff_rod_back_left_joint: origin xyz=-0.04 0.12 0.1875 rpy=0 0 0 -> xyz=-0.055 0.12 0.1875 rpy=0 0 0
- joint standoff_rod_back_right_joint: origin xyz=-0.04 -0.12 0.1875 rpy=0 0 0 -> xyz=-0.055 -0.12 0.1875 rpy=0 0 0
- joint standoff_rod_front_left_joint: origin xyz=0.04 0.12 0.1875 rpy=0 0 0 -> xyz=0.055 0.12 0.1875 rpy=0 0 0
- joint standoff_rod_front_right_joint: origin xyz=0.04 -0.12 0.1875 rpy=0 0 0 -> xyz=0.055 -0.12 0.1875 rpy=0 0 0
