Commit message: Update xacro and RViz configurations

File: xacro/barista_robot_model.urdf.xacro (robot description, xacro)
@@ -93,20 +93,20 @@
     <parent link="chassis"/>
     <child link="standoff_rod_front_left"/>
-    <origin xyz="${tray_diameter/4} ${tray_diameter/4} ${chassis_height/2+standoff_height/2}" rpy="0 0 0"/>
+    <origin xyz="0.055 0.12 0.1875" rpy="0 0 0"/>
 </joint>
 <joint name="standoff_rod_front_right_joint" type="fixed">
     <parent link="chassis"/>
     <child link="standoff_rod_front_right"/>
-    <origin xyz="${tray_diameter/4} ${-tray_diameter/4} ${chassis_height/2+standoff_height/2}" rpy="0 0 0"/>
+    <origin xyz="0.055 -0.12 0.1875" rpy="0 0 0"/>
 </joint>
 <joint name="standoff_rod_back_left_joint" type="fixed">
     <parent link="chassis"/>
     <child link="standoff_rod_back_left"/>
-    <origin xyz="${-tray_diameter/4} ${tray_diameter/4} ${chassis_height/2+standoff_height/2}" rpy="0 0 0"/>
+    <origin xyz="-0.055 0.12 0.1875" rpy="0 0 0"/>
 </joint>
 <joint name="standoff_rod_back_right_joint" type="fixed">
     <parent link="chassis"/>
     <child link="standoff_rod_back_right"/>
-    <origin xyz="${-tray_diameter/4} ${-tray_diameter/4} ${chassis_height/2+standoff_height/2}" rpy="0 0 0"/>
+    <origin xyz="-0.055 -0.12 0.1875" rpy="0 0 0"/>
 </joint>
 <!--chassis and wheels-->
@@ -149,5 +149,5 @@
         <parent link="chassis"/>
         <child link="laser_scanner"/>
-        <origin xyz="${chassis_diameter/3} 0 ${chassis_height/2}" rpy="0 0 0"/>
+        <origin xyz="0.120 0.0 0.1275" rpy="0 0 0"/>
     </joint>
 </xacro:if>
@@ -175,5 +175,5 @@
     <plugin filename="libgazebo_ros_diff_drive.so" name="differential_drive_controller_node">
         <ros>
-            <namespace>/${robot_name}</namespace>
+            <!-- <namespace>/${robot_name}</namespace> -->
             <remapping>/out:=cmd_vel</remapping>
         </ros>

File: xacro/laser_scanner.xacro (robot description, xacro)
@@ -4,7 +4,7 @@
         <xacro:property name="laser_r" value="0.05"/>
         <xacro:property name="laser_h" value="0.07"/>
-        <link name="${name}">
+        <link name="laser_scanner">
             <visual>
-                <origin rpy="0 0 0" xyz="0.0 0.0 0.0"/>
+                <origin rpy="0 0 0" xyz="0.0 0.0 -0.05"/>
                 <geometry>
                     <mesh filename="package://barista_robot_description/meshes/hokuyo_urg_04lx.dae"/>
@@ -12,7 +12,7 @@
             </visual>
             <collision>
-                <origin rpy="0 0 0" xyz="0.0 0.0 0.0"/>
+                <origin rpy="0 0 0" xyz="0.0 0.0 -0.05"/>
                 <geometry>
-                    <mesh filename="package://barista_robot_description/meshes/hokuyo_urg_04lx.dae"/>
+                    <cylinder length="0.040" radius="0.03"/>
                 </geometry>
             </collision>
@@ -26,5 +26,5 @@
         </link>
         <!--laser plugin-->
-        <gazebo reference="${name}">
+        <gazebo reference="laser_scanner">
             <sensor name="sensor_ray" type="ray">
                 <pose>0 0 0 0 0 0</pose>
@@ -51,4 +51,5 @@
                     </ros>
                     <output_type>sensor_msgs/LaserScan</output_type>
+                    <frame_name>laser_scanner</frame_name>
                 </plugin>
             </sensor>

Commit message: Modified xacro for multiple robots

File: xacro/barista_robot_model.urdf.xacro (robot description, xacro)
@@ -4,4 +4,5 @@
 <xacro:property name="robot_name" value="$(arg robot_name)"/>
 <xacro:property name="include_laser" value="$(arg include_laser)"/>
+<xacro:property name="robot_color" default="$(arg robot_color)"/>
 <!--include the macros-->
 <xacro:include filename="$(find barista_robot_description)/xacro/caster_wheel.xacro"/>
@@ -16,25 +17,27 @@
 <xacro:property name="chassis_height" value="0.155"/>
 <xacro:property name="chassis_mass" value="10"/>
-<xacro:property name="chassis_material" value="blue"/>
+<xacro:property name="chassis_material" value="Blue"/>
+<xacro:property name="chassis_gazebo_color" value="Gazebo/Blue"/>
 <!--cup holder tray parameters-->
 <xacro:property name="tray_diameter" value="0.320"/>
 <xacro:property name="tray_height" value="0.090"/>
 <xacro:property name="tray_mass" value="5"/>
-<xacro:property name="tray_material" value="blue"/>
+<xacro:property name="tray_material" value="Blue"/>
+<xacro:property name="tray_gazebo_color" value="Gazebo/Blue"/>
 <!--standoff parameters-->
 <xacro:property name="standoff_diameter" value="0.020"/>
 <xacro:property name="standoff_height" value="0.220"/>
 <xacro:property name="standoff_mass" value="0.2"/>
-<xacro:property name="standoff_material" value="white"/>
+<xacro:property name="standoff_material" value="White"/>
 <!--wheel parameters-->
 <xacro:property name="wheel_diameter" value="0.0704"/>
 <xacro:property name="wheel_width" value="0.0206"/>
 <xacro:property name="wheel_mass" value="0.5"/>
-<xacro:property name="wheel_material" value="black"/>
+<xacro:property name="wheel_material" value="Black"/>
 <xacro:property name="wheel_separation" value="0.300"/>
 <!--caster parameters-->
 <xacro:property name="caster_radius" value="0.020"/>
 <xacro:property name="caster_mass" value="0.1"/>
-<xacro:property name="caster_material" value="black"/>
+<xacro:property name="caster_material" value="Black"/>
 <!--laser parameters-->
 <xacro:property name="laser_mass" value="0.160"/>
@@ -45,11 +48,11 @@
     <color rgba = "1 0 0 0.8 "/>
 </material>
-<material name = "white">
+<material name = "White">
     <color rgba = "1 1 1 1 "/>
 </material>
-<material name = "blue">
+<material name = "Blue">
     <color rgba = "0 0 0.9 0.8 "/>
 </material>
-<material name = "black">
+<material name = "Black">
     <color rgba = "0.1 0.1 0.1 1 "/>
 </material>
@@ -59,6 +62,6 @@
 </link>
 <!--generate the chassis and cup holder tray-->
-<xacro:cup_holder_tray name="chassis" radius="${chassis_diameter/2}" height="${chassis_height}" mass="${chassis_mass}" material="${chassis_material}"/>
-<xacro:cup_holder_tray name="cup_holder_tray" radius="${tray_diameter/2}" height="${tray_height}" mass="${tray_mass}" material="${tray_material}"/>
+<xacro:cup_holder_tray name="chassis" radius="${chassis_diameter/2}" height="${chassis_height}" mass="${chassis_mass}" material="${robot_color}"/>
+<xacro:cup_holder_tray name="cup_holder_tray" radius="${tray_diameter/2}" height="${tray_height}" mass="${tray_mass}" material="${robot_color}"/>
 <!--generate 4 standoff rods-->
 <xacro:standoff_rod name="standoff_rod_front_left" radius="${standoff_diameter/2}" height="${standoff_height}" mass="${standoff_mass}" material="${standoff_material}"/>
@@ -175,5 +178,5 @@
     <plugin filename="libgazebo_ros_diff_drive.so" name="differential_drive_controller_node">
         <ros>
-            <!-- <namespace>/${robot_name}</namespace> -->
+            <namespace>/${robot_name}</namespace>
             <remapping>/out:=cmd_vel</remapping>
         </ros>
@@ -224,8 +227,8 @@
 </gazebo>
 <gazebo reference="chassis">
-    <material>Gazebo/Blue</material>
+    <material>Gazebo/${robot_color}</material>
 </gazebo>
 <gazebo reference="cup_holder_tray">
-    <material>Gazebo/Blue</material>
+    <material>Gazebo/${robot_color}</material>
 </gazebo>
 <gazebo reference="standoff_rod_front_left">

File: xacro/laser_scanner.xacro (robot description, xacro)
@@ -48,4 +48,5 @@
                 <plugin name="laser_scanner_node" filename="libgazebo_ros_ray_sensor.so">
                     <ros>
+                        <namespace>/${robot_name}</namespace>
                         <remapping>~/out:=scan</remapping>
                     </ros>
